File: DigitSynth-Schematic/RPInterface.kicad_sch (KiCad schematic)
At the start: 1 part, among them J1_RPI THD-20-R

Commit message: Add completed KiCad schematic hierarchy (Pi interface, ADC, LEDs, buttons, power)
Parts:
- renumbered J1_RPI to J_RPI1
Connections:
- net +3V3_PI: now also J_RPI1.17 (Pin_17)
Changed lines of the file:
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@@
 	(paper "A4")
+	(junction
+		(at 181.61 35.56)
+		(diameter 0)
+		(color 0 0 0 0)
+	)
 	(junction
 		(at 212.09 76.2)
@@
 	(wire
 		(pts
+			(xy 198.12 55.88) (xy 181.61 55.88)
+		)
+		(stroke
+			(width 0)
+			(type default)
+		)
+	)
+	(wire
+		(pts
 			(xy 173.99 45.72) (xy 196.85 45.72)
 		)
@@
 	(wire
 		(pts
-			(xy 173.99 35.56) (xy 198.12 35.56)
+			(xy 173.99 35.56) (xy 181.61 35.56)
 		)
 		(stroke
@@
 	(wire
 		(pts
+			(xy 181.61 35.56) (xy 198.12 35.56)
+		)
+		(stroke
+			(width 0)
+			(type solid)
+		)
+	)
+	(wire
+		(pts
 			(xy 173.99 71.12) (xy 198.12 71.12)
 		)
@@
 			(width 0)
 			(type solid)
+		)
+	)
+	(wire
+		(pts
+			(xy 181.61 55.88) (xy 181.61 35.56)
+		)
+		(stroke
+			(width 0)
+			(type default)
 		)
 	)
@@
 		(on_board yes)
 		(dnp no)
-		(property "Reference" "J1_RPI"
+		(property "Reference" "J_RPI1"
 			(at 212.09 33.02 0)
 			(effects
@@
 			(project "DigitSynth"
 				(path "/ad908932-4812-48b1-9c87-6bb086cd45d9/91c7c2d9-e939-40fa-a472-fe4cf5507780"
-					(reference "J1_RPI")
+					(reference "J_RPI1")
 					(unit 1)
 				)
