File: DigitSynth-Schematic/RPInterface.kicad_sch (KiCad schematic)
At the start: 1 part

Commit message: KiCad PCB fully routed
Parts:
- added H1, H2, H3, H4: MountingHole, MountingHole:MountingHole_2.7mm_M2.5, symbol Mechanical:MountingHole
