File: DigitSynth-Schematic/ADC_Flex.kicad_sch (KiCad schematic)
At the start: 27 parts, among them J1 Conn_01x02_Pin, J2 Conn_01x02_Pin, J3 Conn_01x02_Pin, J4 Conn_01x02_Pin, U1 ADS1256IDBR

Commit message: KiCad PCB fully routed
Parts:
- C_AVDD_1, C_DVDD_1: footprint (none) -> Capacitor_SMD:C_0603_1608Metric; LCSC Part # (none) -> C14663
- C_AVDD_2: footprint (none) -> Capacitor_SMD:C_0805_2012Metric; LCSC Part # (none) -> C15850
- C_FILT1, C_FILT2, C_FILT3, C_FILT4: footprint (none) -> Capacitor_SMD:C_0603_1608Metric; LCSC Part # (none) -> C1615
- J1, J2, J3, J4: footprint (none) -> Connector_Molex:Molex_KK-254_AE-6410-02A_1x02_P2.54mm_Vertical
- R1, R2, R3, R4: footprint (none) -> Resistor_SMD:R_0603_1608Metric; LCSC Part # (none) -> C21190
- R10, R11, R8, R9: footprint (none) -> Resistor_SMD:R_0603_1608Metric; LCSC Part # (none) -> C22790
- R5, R6, R7: footprint (none) -> Resistor_SMD:R_0603_1608Metric; LCSC Part # (none) -> C25804
- TP1, TP2, TP3, TP4: footprint (none) -> TestPoint:TestPoint_THTPad_D1.0mm_Drill0.5mm
- U1: footprint ADS1256IDBR:SOP65P780X200-28N -> Package_SO:SSOP-28_5.3x10.2mm_P0.65mm; Availability In Stock -> (none); Check_prices https://www.snapeda.com/parts/ADS1256IDBR/Texas+Instruments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 -> (none); LCSC Part # (none) -> C28186; Price None -> (none); Purchase-URL https://www.snapeda.com/api/url_track_click_mouser/?unipart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 -> (none); SnapEDA_Link https://www.snapeda.com/parts/ADS1256IDBR/Texas+Instruments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 -> (none)
