File: DigitSynth-Schematic/DigitSynth.kicad_sch (KiCad schematic)
At the start: 0 parts

Commit message: KiCad PCB fully routed
Other:
- sheet ADC Flex ports: added none; removed FLEX1_V, FLEX2_V, FLEX3_V, FLEX4_V
Changed lines of the file:
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@@
-			)
-		)
-		(pin "FLEX1_V" output
-			(at 91.44 118.11 180)
-			(effects
-				(font
-					(size 1.27 1.27)
-				)
-				(justify left)
-			)
-		)
-		(pin "FLEX2_V" output
-			(at 91.44 113.03 180)
-			(effects
-				(font
-					(size 1.27 1.27)
-				)
-				(justify left)
-			)
-		)
-		(pin "FLEX3_V" output
-			(at 91.44 107.95 180)
-			(effects
-				(font
-					(size 1.27 1.27)
-				)
-				(justify left)
-			)
-		)
-		(pin "FLEX4_V" output
-			(at 91.44 104.14 180)
-			(effects
-				(font
-					(size 1.27 1.27)
-				)
-				(justify left)
 			)
 		)
